Commit message: solving slitting problem

File: description/robot_core.xacro (robot description, xacro)
@@ -64,5 +64,6 @@
         <collision> <!-- physic collision -->
             <geometry>
-                <cylinder radius="0.05" length="0.04"/> <!-- same as visual-->
+                <sphere radius = "0.05"/>
+                <!-- <cylinder radius="0.05" length="0.04"/>  same as visual-->
             </geometry>
         </collision>
@@ -90,5 +91,6 @@
         <collision> <!-- physic collision -->
             <geometry>
-                <cylinder radius="0.05" length="0.04"/> <!-- same as visual-->
+                <sphere radius = "0.05"/>
+                <!-- <cylinder radius="0.05" length="0.04"/>  same as visual-->
             </geometry>
         </collision>

File: description/ros2_control.xacro (robot description, xacro)
@@ -24,5 +24,5 @@
     <gazebo>
         <plugin name="gazebo_ros2_control" filename="libgazebo_ros2_control.so">
-            <parameters>$(find my_bot)/config/my_controllers.yaml</parameters>
+            <parameters>$(find tizio_bot)/config/my_controllers.yaml</parameters>
         </plugin>
     </gazebo>
